Commit message: Update files

File: src/my_robot/urdf/my_robot.urdf (robot description, URDF)
Before this commit: robot ece2318_robot, 12 links, 11 joints
Links:
- added link camera_lens, mass 0.05; visual cylinder length=0.04 radius=0.045
- added link camera_link, mass 0.2; collision box size=0.12 0.32 0.1; visual box size=0.12 0.32 0.1
- added link imu_link, mass 0.05; visual box size=0.05 0.05 0.02
- added link left_fingertip, mass 0.02; visual sphere radius=0.05
- added link lidar_ring, mass 0.1; visual cylinder length=0.04 radius=0.24
- added link right_fingertip, mass 0.02; visual sphere radius=0.05
- added link status_led, mass 0.01; visual sphere radius=0.07
- added link top_panel, mass 2.0; visual box size=2.8 1.8 0.05
- added link wrist_link, mass 0.8; collision cylinder length=0.12 radius=0.12; visual cylinder length=0.12 radius=0.12
- link arm_base: mass None -> 4.0; geometry collision cylinder length=0.22 radius=0.36; visual cylinder length=0.22 radius=0.36
- link arm_link_1: mass None -> 5.0; geometry collision box size=0.28 0.28 1.6; visual box size=0.28 0.28 1.6
- link arm_link_2: mass None -> 3.0; geometry collision box size=0.22 0.22 1.2; visual box size=0.22 0.22 1.2
- link base_link: mass None -> 60.0; geometry collision box size=3.0 2.0 0.9; visual box size=3.0 2.0 0.9
- link front_left_wheel: mass None -> 3.0; geometry collision cylinder length=0.38 radius=0.55; visual cylinder length=0.38 radius=0.55
- link front_right_wheel: mass None -> 3.0; geometry collision cylinder length=0.38 radius=0.55; visual cylinder length=0.38 radius=0.55
- link gripper_base: mass None -> 0.5; geometry collision box size=0.45 0.18 0.12; visual box size=0.45 0.18 0.12
- link left_finger: mass None -> 0.15; geometry collision box size=0.09 0.09 0.44; visual box size=0.09 0.09 0.44
- link lidar_link: mass None -> 0.5; geometry collision cylinder length=0.14 radius=0.22; visual cylinder length=0.14 radius=0.22
- link rear_left_wheel: mass None -> 3.0; geometry collision cylinder length=0.38 radius=0.55; visual cylinder length=0.38 radius=0.55
- link rear_right_wheel: mass None -> 3.0; geometry collision cylinder length=0.38 radius=0.55; visual cylinder length=0.38 radius=0.55
- link right_finger: mass None -> 0.15; geometry collision box size=0.09 0.09 0.44; visual box size=0.09 0.09 0.44
Joints:
- added joint camera_joint: type fixed, parent base_link, child camera_link, origin xyz=1.52 0 0.15 rpy=0 0 0
- added joint camera_lens_joint: type fixed, parent camera_link, child camera_lens, origin xyz=0.08 0 0 rpy=0 1.5708 0
- added joint gripper_base_joint: type fixed, parent wrist_link, child gripper_base, origin xyz=0 0 0.12 rpy=0 0 0
- added joint imu_joint: type fixed, parent base_link, child imu_link, origin xyz=0 0 0.46 rpy=0 0 0
- added joint left_fingertip_joint: type fixed, parent left_finger, child left_fingertip, origin xyz=0 0 0.46 rpy=0 0 0
- added joint lidar_ring_joint: type fixed, parent lidar_link, child lidar_ring, origin xyz=0 0 -0.09 rpy=0 0 0
- added joint right_fingertip_joint: type fixed, parent right_finger, child right_fingertip, origin xyz=0 0 0.46 rpy=0 0 0
- added joint status_led_joint: type fixed, parent base_link, child status_led, origin xyz=-1.3 0.0 0.5 rpy=0 0 0
- added joint top_panel_joint: type fixed, parent base_link, child top_panel, origin xyz=0 0 0.475 rpy=0 0 0
- joint arm_base_joint: limit (none) -> lower=-3.14159 upper=3.14159 effort=50 velocity=1.0; origin xyz=0.0 0 0.6 rpy=0 0 0 -> xyz=0.0 0 0.56 rpy=0 0 0; type continuous -> revolute
- joint elbow_joint: limit (none) -> lower=-2.0944 upper=0.0 effort=60 velocity=1.0; type continuous -> revolute
- joint fl_wheel_joint: origin xyz=1.0 1.2 -0.5 rpy=1.5708 0 0 -> xyz=1.0 1.2 -0.45 rpy=1.5708 0 0
- joint fr_wheel_joint: origin xyz=1.0 -1.2 -0.5 rpy=1.5708 0 0 -> xyz=1.0 -1.2 -0.45 rpy=1.5708 0 0
- joint left_finger_joint: limit lower=0 upper=0.1 effort=10 velocity=0.5 -> lower=0.0 upper=0.18 effort=20 velocity=0.5; origin xyz=0.2 0 0.1 rpy=0 0 0 -> xyz=0.18 0 0.06 rpy=0 0 0
- joint lidar_joint: origin xyz=1.3 0 0.75 rpy=0 0 0 -> xyz=1.2 0 0.55 rpy=0 0 0
- joint right_finger_joint: limit lower=0 upper=0.1 effort=10 velocity=0.5 -> lower=0.0 upper=0.18 effort=20 velocity=0.5; origin xyz=-0.2 0 0.1 rpy=0 0 0 -> xyz=-0.18 0 0.06 rpy=0 0 0
- joint rl_wheel_joint: origin xyz=-1.0 1.2 -0.5 rpy=1.5708 0 0 -> xyz=-1.0 1.2 -0.45 rpy=1.5708 0 0
- joint rr_wheel_joint: origin xyz=-1.0 -1.2 -0.5 rpy=1.5708 0 0 -> xyz=-1.0 -1.2 -0.45 rpy=1.5708 0 0
- joint shoulder_joint: limit (none) -> lower=-1.5708 upper=1.5708 effort=80 velocity=0.8; origin xyz=0 0 0.1 rpy=0 0 0 -> xyz=0 0 0.11 rpy=0 0 0; type continuous -> revolute
- joint wrist_joint: child gripper_base -> wrist_link; limit (none) -> lower=-1.5708 upper=1.5708 effort=30 velocity=1.5; type continuous -> revolute

Commit message: Update files

File: src/my_robot/urdf/my_robot.urdf (robot description, URDF)
Before this commit: robot ece2318_robot, 21 links, 20 joints
Joints:
- joint fr_wheel_joint: origin xyz=1.0 -1.2 -0.45 rpy=1.5708 0 0 -> xyz=1.0 -1.2 -0.45 rpy=-1.5708 0 0
- joint rr_wheel_joint: origin xyz=-1.0 -1.2 -0.45 rpy=1.5708 0 0 -> xyz=-1.0 -1.2 -0.45 rpy=-1.5708 0 0
